Commit message: Add files via upload

File: urdf/robot.xacro (robot description, xacro)
@@ -1,102 +1,68 @@
-<?xml version="1.0" ?>
-<robot name="navvis">
-  <link name="base">
-    <visual>
-      <origin rpy="0.0 0.0 0.0" xyz="0.0 0.0 0.96"/>
-      <geometry>
-        <box size="0.45 0.78 1.92"/>
-      </geometry>
-    </visual>
-    <collision>
-      <origin rpy="0.0 0.0 0.0" xyz="0.0 0.0 0.96"/>
-      <geometry>
-        <box size="0.45 0.78 1.92"/>
-      </geometry>
-    </collision>
-  </link>
-  <link name="laser_vert_bottom">
-    <visual>
-      <geometry>
-        <box size="0.062 0.062 0.087"/>
-      </geometry>
-    </visual>
-    <collision>
-      <geometry>
-        <box size="0.062 0.062 0.087"/>
-      </geometry>
-    </collision>
-  </link>
-  <link name="laser_vert_top_right">
-    <visual>
-      <geometry>
-        <box size="0.062 0.062 0.087"/>
-      </geometry>
-    </visual>
-    <collision>
-      <geometry>
-        <box size="0.062 0.062 0.087"/>
-      </geometry>
-    </collision>
-  </link>
-  <link name="laser_vert_top_left">
-    <visual>
-      <geometry>
-        <box size="0.062 0.062 0.087"/>
-      </geometry>
-    </visual>
-    <collision>
-      <geometry>
-        <box size="0.062 0.062 0.087"/>
-      </geometry>
-    </collision>
-  </link>
-  <link name="laser_horiz">
-    <visual>
-      <geometry>
-        <cylinder length="0.072" radius="0.052"/>
-      </geometry>
-    </visual>
-    <collision>
-      <geometry>
-        <cylinder length="0.072" radius="0.052"/>
-      </geometry>
-    </collision>
-  </link>
-  <joint name="base_laser_vert_bottom_joint" type="fixed">
-    <parent link="base"/>
-    <child link="laser_vert_bottom"/>
-    <origin rpy="3.1355 -1.3045 0.0025" xyz="0.3158 -0.0021 0.51"/>
-  </joint>
-  <joint name="base_laser_vert_top_right_joint" type="fixed">
-    <parent link="base"/>
-    <child link="laser_vert_top_right"/>
-    <origin rpy="-1.1760 0.6313 -1.9377" xyz="0.2978 -0.1450 1.8451"/>
-  </joint>
-  <joint name="base_laser_vert_top_left_joint" type="fixed">
-    <parent link="base"/>
-    <child link="laser_vert_top_left"/>
-    <origin rpy="1.1780 0.6198 1.9560" xyz="0.2997 0.1531 1.8443"/>
-  </joint>
-  <joint name="base_laser_horiz_joint" type="fixed">
-    <parent link="base"/>
-    <child link="laser_horiz"/>
-    <origin rpy="-0.0012 0.1146 -0.0015" xyz="0.2325 0.0001 1.9201"/>
-  </joint>
-  <link name="wheel_left">
-    <visual>
-      <geometry>
-        <cylinder length="0.05" radius="0.2"/>
-      </geometry>
-    </visual>
-    <collision>
-      <geometry>
-        <cylinder length="0.05" radius="0.2"/>
-      </geometry>
-    </collision>
-  </link>
-  <joint name="base_wheel_left_joint" type="fixed">
-    <parent link="base"/>
-    <child link="wheel_left"/>
-    <origin rpy="-1.57 0 0" xyz="-0.1 0.4 0"/>
-  </joint>
+<?xml version="1.0"?>
+<robot xmlns:xacro="http://www.ros.org/wiki/xacro" name="navvis">
+	<link name="base">
+		<visual>
+			<origin xyz="0.0 0.0 0.96" rpy="0.0 0.0 0.0" />
+			<geometry>
+				<box size="0.45 0.78 1.92" />
+			</geometry>
+		</visual>
+		<collision>
+			<origin xyz="0.0 0.0 0.96" rpy="0.0 0.0 0.0" />
+			<geometry>
+				<box size="0.45 0.78 1.92" />
+			</geometry>
+		</collision>
+	</link>
+	<xacro:include filename="$(find gazebo_plugins)/test/multi_robot_scenario/xacro/laser/hokuyo.xacro" />
+	<xacro:include filename="$(find velodyne_description)/urdf/VLP-16.urdf.xacro"/>
+	<xacro:laser name="laser_vert_bottom" parent="base" xyz="0.3158 -0.0021 0.51" rpy="3.1355 -1.3045 0.0025"
+	meshes="package://gazebo_plugins/test/multi_robot_scenario/meshes/laser" />
+	<xacro:laser name="laser_vert_top_right" parent="base" xyz="0.2978 -0.1450 1.8451" rpy="-1.1760 0.6313 -1.9377"
+	meshes="package://gazebo_plugins/test/multi_robot_scenario/meshes/laser" />
+	<xacro:laser name="laser_vert_top_left" parent="base" xyz="0.2997 0.1531 1.8443" rpy="1.1780 0.6198 1.9560"
+	meshes="package://gazebo_plugins/test/multi_robot_scenario/meshes/laser" />
+	<xacro:VLP-16 parent="base" name="laser_horiz" topic="laser_horiz/packets" hz="10" samples="440" gpu="false">
+		<origin xyz="0.2325 0.0001 1.9201" rpy="-0.0012 0.1146 -0.0015" />
+	</xacro:VLP-16>
+	<xacro:macro name="xacro_name" params="side reflect">
+		<link name="wheel_${side}">
+			<visual>
+				<geometry>
+					<cylinder length="0.05" radius="0.2" />
+				</geometry>
+			</visual>
+			<collision>
+				<geometry>
+					<cylinder length="0.05" radius="0.2" />
+				</geometry>
+			</collision>
+		</link>
+		<joint name="base_wheel_${side}_joint" type="continuous">
+			<parent link="base" />
+			<child link="wheel_${side}" />
+			<origin xyz="-0.1 ${reflect * 0.4} 0" rpy="-1.57 0 0" />
+			<axis xyz="0 0 1" />
+		</joint>
+	</xacro:macro>
+	<xacro:xacro_name side="left" reflect="1" />
+	<xacro:xacro_name side="right" reflect="-1" />
+	<link name="wheel_center">
+		<visual>
+			<geometry>
+				<cylinder length="0.05" radius="0.15" />
+			</geometry>
+		</visual>
+		<collision>
+			<geometry>
+				<cylinder length="0.05" radius="0.15" />
+			</geometry>
+		</collision>
+	</link>
+	<joint name="base_wheel_center_joint" type="continuous">
+		<parent link="base" />
+		<child link="wheel_center" />
+		<origin xyz="0.1 0 -0.05" rpy="-1.57 0 0" />
+		<axis xyz="0 0 1" />
+	</joint>
 </robot>
